Commit message: single and bimanual arms in gazebo, isac sim bridge and bimanual arms in isaacsim

File: src/lerobot_description/urdf/bi_so101_isaac.urdf.xacro (robot description, xacro)
@@ -1,10 +1,11 @@
 <?xml version="1.0"?>
 <!--
-  Bimanual SO-101 Robot
-  This file creates a bimanual SO-101 robot by instantiating two SO-101 arms
-  with "left_" and "right_" prefixes. The arms are mounted on a shared table/base
-  with symmetric positioning.
+  Bimanual SO-101 Robot with Isaac Sim Integration
+  This file creates a bimanual SO-101 robot configured for Isaac Sim.
+  It uses topic_based_ros2_control to bridge between Isaac Sim and ROS2.
+  Isaac Sim handles the actual physics simulation and publishes joint states.
+  This URDF is used by robot_state_publisher and ros2_control on the ROS2 side.
 -->
-<robot name="bi_so101" xmlns:xacro="http://www.ros.org/wiki/xacro">
+<robot name="bi_so101_isaac" xmlns:xacro="http://www.ros.org/wiki/xacro">
 	<!-- Configurable Parameters -->
 	<!-- Distance of each arm from table center along X-axis (meters) -->
@@ -12,6 +13,6 @@
 	<!-- Include SO-101 arm macro -->
 	<xacro:include filename="$(find lerobot_description)/urdf/so101_macro.xacro" />
-	<!-- Include ROS2 Control (includes Gazebo plugins) -->
-	<xacro:include filename="$(find lerobot_description)/urdf/bi_so101_ros2_control.xacro" />
+	<!-- Include Isaac Sim ROS2 Control -->
+	<xacro:include filename="$(find lerobot_description)/urdf/bi_so101_isaac_ros2_control.xacro" />
 	<!-- World link (fixed reference frame) -->
 	<link name="world" />

File: src/lerobot_description/urdf/so101.urdf.xacro (robot description, xacro)
@@ -1,6 +1,18 @@
 <?xml version="1.0"?>
+<!--
+  Single SO-101 Robot Arm
+  This file creates a single SO-101 robot arm by instantiating the SO-101 arm macro
+  with no prefix. The arm is mounted on a world reference frame.
+-->
 <robot name="so101" xmlns:xacro="http://www.ros.org/wiki/xacro">
-    <xacro:include filename="$(find lerobot_description)/urdf/so101_base.xacro" />
-    <xacro:include filename="$(find lerobot_description)/urdf/so101_gazebo.xacro" />
-    <xacro:include filename="$(find lerobot_description)/urdf/so101_ros2_control.xacro" />
+	<!-- Include SO-101 arm macro -->
+	<xacro:include filename="$(find lerobot_description)/urdf/so101_macro.xacro" />
+	<!-- Include ROS2 Control -->
+	<xacro:include filename="$(find lerobot_description)/urdf/so101_ros2_control.xacro" />
+	<!-- World link (fixed reference frame) -->
+	<link name="world" />
+	<!-- Single arm - instantiate macro with no prefix -->
+	<xacro:so101_arm prefix="" parent="world">
+		<origin xyz="0 0 0" rpy="0 0 0" />
+	</xacro:so101_arm>
 </robot>

File: src/lerobot_description/urdf/so101_macro.xacro (robot description, xacro)
@@ -9,5 +9,5 @@
 	<!-- Materials (shared across all instances) -->
 	<material name="3d_printed">
-		<color rgba="1.0 0.82 0.12 1.0" />
+		<color rgba="0.12 0.12 0.12 1.0" />
 	</material>
 	<material name="sts3215">

File: src/lerobot_description/urdf/so101_ros2_control.xacro (robot description, xacro)
@@ -49,3 +49,9 @@
         </joint>
     </ros2_control>
+    <!-- Gazebo ROS2 Control plugin -->
+    <gazebo>
+        <plugin filename="gz_ros2_control-system" name="gz_ros2_control::GazeboSimROS2ControlPlugin">
+            <parameters>$(find lerobot_controller)/config/so101_controllers.yaml</parameters>
+        </plugin>
+    </gazebo>
 </robot>
